File: PCB Files/PCB.kicad_pcb (KiCad board)
At the start: 2 copper layers, 94 x 80 mm, 19 parts, among them M1 Conn_01x02_Pin, M2 Conn_01x02_Pin, M3 Conn_01x02_Pin, M4 Conn_01x02_Pin

Commit message: Updated PCB Files
Connections:
- A1 pad 27: unconnected-(A1-+5V-Pad27) -> 5V
- ESC1 pad 2: unconnected-(ESC1-Pin_2-Pad2) -> 5V
- ESC2 pad 2: unconnected-(ESC2-Pin_2-Pad2) -> 5V
- ESC3 pad 2: unconnected-(ESC3-Pin_2-Pad2) -> 5V
- ESC4 pad 2: unconnected-(ESC4-Pin_2-Pad2) -> 5V
- GY91 pad 1: unconnected-(GY91-Pin_1-Pad1) -> 5V
- InputPower1 pad 2: unconnected-(InputPower1-Pin_2-Pad2) -> 5V
- LED_Builtin1 pad 2: unconnected-(LED_Builtin1-A-Pad2) -> 5V
- On/Off1 pad 2: unconnected-(On/Off1-A-Pad2) -> 5V
- Power1 pad 1: unconnected-(Power1-Pin_1-Pad1) -> 5V
- Power1 pad 3: unconnected-(Power1-Pin_3-Pad3) -> 5V
- Power1 pad 5: unconnected-(Power1-Pin_5-Pad5) -> 5V
Routing:
- net GND: track 0.00 -> 347.7 mm
- net 5V: track 0.00 -> 270.4 mm
- net +BATT: track 0.00 -> 147.6 mm
- net Net-(A1-D7): track 0.00 -> 90.7 mm
- net Net-(A1-D6): track 0.00 -> 73.1 mm
- net Net-(A1-A5): track 0.00 -> 70.7 mm
- net Net-(A1-A6): track 0.00 -> 67.4 mm
- net Net-(A1-A1): track 0.00 -> 67.3 mm
- net Net-(A1-D5): track 0.00 -> 66.6 mm
- net Net-(A1-A4): track 0.00 -> 64.6 mm
- net Net-(A1-D4): track 0.00 -> 60.0 mm
- net Net-(A1-A3): track 0.00 -> 52.8 mm
- net Net-(A1-A0): track 0.00 -> 51.5 mm
- net Net-(A1-A2): track 0.00 -> 47.2 mm
- net Net-(A1-D0/RX): track 0.00 -> 36.8 mm
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