File: PCB Files/PCB.kicad_sch (KiCad schematic)
At the start: 19 parts, among them M1 Conn_01x02_Pin, M2 Conn_01x02_Pin, M3 Conn_01x02_Pin, M4 Conn_01x02_Pin

Commit message: Updated PCB Files
Connections:
- net 5V: now also A1.27 (+5V), ESC1.2 (Pin_2), ESC2.2 (Pin_2), ESC3.2 (Pin_2), ESC4.2 (Pin_2), GY91.1 (Pin_1), InputPower1.2 (Pin_2), LED_Builtin1.2 (A), On/Off1.2 (A), Power1.1 (Pin_1), Power1.3 (Pin_3), Power1.5 (Pin_5)
Changed lines of the file:
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@@
 	(wire
 		(pts
-			(xy 31.75 86.36) (xy 31.75 74.93)
+			(xy 156.21 93.98) (xy 161.29 93.98)
 		)
 		(stroke
@@
 	(wire
 		(pts
+			(xy 165.1 54.61) (xy 170.18 54.61)
+		)
+		(stroke
+			(width 0)
+			(type default)
+		)
+	)
+	(wire
+		(pts
 			(xy 143.51 38.1) (xy 92.71 38.1)
 		)
@@
 	(wire
 		(pts
+			(xy 173.99 22.86) (xy 173.99 27.94)
+		)
+		(stroke
+			(width 0)
+			(type default)
+		)
+	)
+	(wire
+		(pts
 			(xy 57.15 96.52) (xy 57.15 85.09)
 		)
@@
 	(wire
 		(pts
-			(xy 31.75 74.93) (xy 19.05 74.93)
+			(xy 146.05 22.86) (xy 146.05 27.94)
 		)
 		(stroke
@@
 	(wire
 		(pts
+			(xy 25.4 129.54) (xy 30.48 129.54)
+		)
+		(stroke
+			(width 0)
+			(type default)
+		)
+	)
+	(wire
+		(pts
 			(xy 243.84 116.84) (xy 243.84 95.25)
 		)
@@
 	(wire
 		(pts
-			(xy 113.03 86.36) (xy 31.75 86.36)
-		)
-		(stroke
-			(width 0)
-			(type default)
-		)
-	)
-	(wire
-		(pts
 			(xy 46.99 93.98) (xy 46.99 82.55)
 		)
@@
 	(wire
 		(pts
+			(xy 25.4 134.62) (xy 30.48 134.62)
+		)
+		(stroke
+			(width 0)
+			(type default)
+		)
+	)
+	(wire
+		(pts
 			(xy 19.05 82.55) (xy 46.99 82.55)
 		)
@@
 	(wire
 		(pts
+			(xy 111.76 86.36) (xy 113.03 86.36)
+		)
+		(stroke
+			(width 0)
+			(type default)
+		)
+	)
+	(wire
+		(pts
 			(xy 113.03 104.14) (xy 96.52 104.14)
 		)
@@
 	(wire
 		(pts
+			(xy 130.81 71.12) (xy 130.81 76.2)
+		)
+		(stroke
+			(width 0)
+			(type default)
+		)
+	)
+	(wire
+		(pts
+			(xy 269.24 115.57) (xy 274.32 115.57)
+		)
+		(stroke
+			(width 0)
+			(type default)
+		)
+	)
+	(wire
+		(pts
 			(xy 142.24 106.68) (xy 142.24 66.04)
 		)
@@
 	(wire
 		(pts
+			(xy 25.4 139.7) (xy 30.48 139.7)
+		)
+		(stroke
+			(width 0)
+			(type default)
+		)
+	)
+	(wire
+		(pts
 			(xy 204.47 104.14) (xy 204.47 90.17)
 		)
@@
 	(wire
 		(pts
+			(xy 19.05 74.93) (xy 111.76 74.93)
+		)
+		(stroke
+			(width 0)
+			(type default)
+		)
+	)
+	(wire
+		(pts
 			(xy 139.7 101.6) (xy 139.7 62.23)
 		)
@@
 	(wire
 		(pts
+			(xy 156.21 22.86) (xy 156.21 27.94)
+		)
+		(stroke
+			(width 0)
+			(type default)
+		)
+	)
+	(wire
+		(pts
 			(xy 162.56 40.64) (xy 95.25 40.64)
 		)
@@
 	(wire
 		(pts
+			(xy 165.1 22.86) (xy 165.1 27.94)
+		)
+		(stroke
+			(width 0)
+			(type default)
+		)
+	)
+	(wire
+		(pts
 			(xy 93.98 99.06) (xy 62.23 99.06)
 		)
@@
 		(pts
 			(xy 92.71 38.1) (xy 92.71 96.52)
+		)
+		(stroke
+			(width 0)
+			(type default)
+		)
+	)
+	(wire
+		(pts
+			(xy 168.91 82.55) (xy 173.99 82.55)
+		)
+		(stroke
+			(width 0)
+			(type default)
+		)
+	)
+	(wire
+		(pts
+			(xy 111.76 74.93) (xy 111.76 86.36)
 		)
 		(stroke
@@
 			(effects
 				(font
+					(size 1.27 1.27)
+				)
+				(justify right)
+				(hide yes)
+			)
+		)
+	)
+	(global_label "5V"
+		(shape output)
+		(at 173.99 82.55 180)
+		(fields_autoplaced yes)
+		(effects
+			(font
+				(size 1.27 1.27)
+				(thickness 0.254)
+				(bold yes)
+			)
+			(justify right)
+		)
+		(property "Intersheetrefs" "${INTERSHEET_REFS}"
+			(at 168.2307 82.55 0)
+			(effects
+				(font
